Commit message: Added gazebo plugins

File: src/blacksail_description/urdf/blacksail_description.urdf (robot description, URDF)
Before this commit: robot blacksail_description, 6 links, 5 joints
Joints:
- joint hull_left_cam: axis 0 0 0 -> 0 1 0; limit (none) -> lower=-1.57 upper=1.57 effort=0 velocity=0; type fixed -> revolute

File: src/blacksail_gazebo/gazebo/asv.xacro (robot description, xacro)
@@ -2,17 +2,6 @@
 <!-- Includes all macros in this package so they don't need to be included individualy -->
 <robot xmlns:xacro="http://ros.org/wiki/xacro"
-       name="WAM-V">
+       name="Blacksail">
   <!-- Include dynamics macros -->
-  <xacro:include filename="$(find wamv_gazebo)/urdf/dynamics/wamv_gazebo_dynamics_plugin.xacro" />
-  <!-- Include sensor macros -->
-  <xacro:include filename="$(find wamv_gazebo)/urdf/sensors/wamv_camera.xacro" />
-  <xacro:include filename="$(find wamv_gazebo)/urdf/sensors/wamv_gps.xacro" />
-  <xacro:include filename="$(find wamv_gazebo)/urdf/sensors/wamv_imu.xacro" />
-  <xacro:include filename="$(find wamv_gazebo)/urdf/sensors/wamv_planar_lidar.xacro" />
-  <xacro:include filename="$(find wamv_gazebo)/urdf/sensors/wamv_3d_lidar.xacro" />
-  <xacro:include filename="$(find wamv_gazebo)/urdf/sensors/lidar.xacro" />
-  <xacro:include filename="$(find wamv_gazebo)/urdf/sensors/wamv_p3d.xacro" />
-  <xacro:include filename="$(find wamv_gazebo)/urdf/sensors/wamv_pinger.xacro" />
-  <!-- Include ball shooter macros -->
-  <xacro:include filename="$(find wamv_gazebo)/urdf/ball_shooter/ball_shooter.xacro" />
+  <xacro:include filename="$(find blacksail_description)/urdf/blacksail_description.urdf" />
 </robot>
